Commit message: update

File: models/rover/model.urdf (robot description, URDF)
Before this commit: robot rover, 13 links, 12 joints
Joints:
- joint wheel_1_joint: axis 0 0 1 -> 0 0 -1
- joint wheel_2_joint: axis 0 0 1 -> 0 0 -1
- joint wheel_3_joint: axis 0 0 1 -> 0 0 -1

Commit message: prototyping

File: models/rover/model.urdf (robot description, URDF)
Before this commit: robot rover, 13 links, 12 joints
Joints:
- joint left_boggie_joint: limit (none) -> lower=-1.047 upper=1.047 effort=1000.0 velocity=1.5707; type continuous -> revolute
- joint left_handle_joint: limit (none) -> lower=-1.047 upper=1.047 effort=1000.0 velocity=1.5707; type continuous -> revolute
- joint right_boggie_joint: limit (none) -> lower=-1.047 upper=1.047 effort=1000.0 velocity=1.5707; type continuous -> revolute
- joint right_handle_joint: limit (none) -> lower=-1.047 upper=1.047 effort=1000.0 velocity=1.5707; type continuous -> revolute

Commit message: improvements

File: models/rover/model.urdf (robot description, URDF)
Before this commit: robot rover, 13 links, 12 joints
Joints:
- joint wheel_1_joint: origin xyz=0.264321 -0.213856  0.132 rpy=0 0 0 -> xyz=0.264321 -0.213856 0.132 rpy=0 0 0
